File: payoad_board.kicad_sch (KiCad schematic)
At the start: 3 parts, among them J1 NMHH-1_bus, U3 RP2040 MCU board, U4 RP2040 MCU board

Commit message: Project libraries, PQ_bus connector symbol, CAN2 on the bus
- Add project-local symbol (pq.kicad_sym) and footprint library tables,
  both relative to ${KIPRJMOD}, so the project opens without extra setup
- New PQ_bus symbol: supply pins are power outputs, so ERC passes
  without PWR_FLAGs; replaces the generic 2x8 connector
- Bus connector footprint renamed to PQ_bus, 3D model assigned
- CAN2 routed to bus pins 6/8 (U2); CAN1 on pins 9/11 (U1)
- 1-Wire notes on the schematic, MCUs re-annotated to U1/U2
- README: PQ_bus pinout with DNC pins, library and file list

Co-Authored-By: Claude Opus 5.5 <noreply@anthropic.com>
Parts:
- removed J1: NMHH-1_bus, pq:PinHeader_2x8_2.54_PCB_edge, symbol Connector_Generic:Conn_02x08_Odd_Even
- added J1: PQ_bus, pq:PinHeader_2x8_2.54_PCB_edge, symbol pq:PQ_bus
- renumbered U3 to U1, U4 to U2
Connections:
- net +3V3: now also J1.7 (REG_BUS_PROTECTED_1)
- net 1W_1: now also J1.13 (1W_1)
- net 1W_2: now also J1.4 (1W_2)
- net CAN1_H: now also J1.11 (CAN1_H)
- net CAN1_L: now also J1.9 (CAN1_L)
- net CAN2_H: now also J1.6 (CAN2_H)
- net CAN2_L: now also J1.8 (CAN2_L)
- net GND: now also J1.1 (GND), J1.16 (GND)
- net VCC: now also J1.10 (REG_BUS_PROTECTED_2)
Other:
- note added: "If 1W_1 is used DO NOT CONNECT anything to GPIO4 ->"
- note added: "If 1W_2 is used DO NOT CONNECT anything to GPIO0 ->"
- moved on the sheet: U1, U2
