File: payoad_board.kicad_sch (KiCad schematic)
At the start: 3 parts, among them J1 PQ_bus, U1 RP2040 MCU board, U2 RP2040 MCU board

Commit message: Rename 1W/1-Wire signals to HDUART
1-Wire is a trademarked name, so the bus signals and MCU pin labels
are now called HDUART (HDUART_1, HDUART_2, GPIO05/HDUART1, ...).

Co-Authored-By: Claude Opus 5.5 <noreply@anthropic.com>
Connections:
- net 1W_1 renamed HDUART_1
- net 1W_2 renamed HDUART_2
Other:
- note added: "If HDUART_1 is used DO NOT CONNECT anything to GPIO4 ->"
- note added: "If HDUART_2 is used DO NOT CONNECT anything to GPIO0 ->"
- note removed: "If 1W_1 is used DO NOT CONNECT anything to GPIO4 ->"
- note removed: "If 1W_2 is used DO NOT CONNECT anything to GPIO0 ->"
Changed lines of the file:
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@@
 		)
 	)
-	(text "If 1W_2 is used DO NOT CONNECT anything to GPIO0 ->"
+	(text "If HDUART_2 is used DO NOT CONNECT anything to GPIO0 ->"
 		(exclude_from_sim no)
 		(at 105.156 111.506 0)
@@
 		)
 	)
-	(text "If 1W_1 is used DO NOT CONNECT anything to GPIO4 ->"
+	(text "If HDUART_1 is used DO NOT CONNECT anything to GPIO4 ->"
 		(exclude_from_sim no)
 		(at 105.41 49.276 0)
@@
 		)
 	)
-	(global_label "1W_1"
+	(global_label "HDUART_1"
 		(shape input)
 		(at 48.26 54.61 180)
@@
 		)
 	)
-	(global_label "1W_2"
+	(global_label "HDUART_2"
 		(shape input)
 		(at 60.96 41.91 0)
@@
 		)
 	)
-	(global_label "1W_2"
+	(global_label "HDUART_2"
 		(shape input)
 		(at 162.56 113.03 180)
@@
 		)
 	)
-	(global_label "1W_1"
+	(global_label "HDUART_1"
 		(shape input)
 		(at 162.56 50.8 180)
